File: KiCad/v2/tiny/panic_button_tiny/panic_button_tiny.kicad_sch (KiCad schematic)
At the start: 0 parts

Commit message: [UPDATE] some connections in the schematic
Other:
- added sheet Visual (visual.kicad_sch)
- sheet brains ports: added LED DIN, UART (RXD), UART (TXD), battery_voltage_sense; removed AT UART (RXD), AT UART (TXD), Battery_voltage_sense
- sheet network_and_gps ports: added UART (RXD), UART (TXD), power-on_pulse; removed UART RXD, UART TXD, power_on_pulse
Changed lines of the file:
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@@
+	(wire
+		(pts
+			(xy 209.55 106.68) (xy 199.39 106.68)
+		)
+		(stroke
+			(width 0)
+			(type default)
+		)
+	)
 	(wire
 		(pts
@@
 	(wire
 		(pts
+			(xy 215.9 116.84) (xy 209.55 116.84)
+		)
+		(stroke
+			(width 0)
+			(type default)
+		)
+	)
+	(wire
+		(pts
 			(xy 139.7 67.31) (xy 139.7 78.74)
 		)
@@
 		(pts
 			(xy 135.89 76.2) (xy 137.16 76.2)
+		)
+		(stroke
+			(width 0)
+			(type default)
+		)
+	)
+	(wire
+		(pts
+			(xy 209.55 116.84) (xy 209.55 106.68)
 		)
 		(stroke
@@
 			)
 		)
-		(pin "UART RXD" input
+		(pin "UART (RXD)" input
 			(at 134.62 67.31 270)
 			(effects
@@
 			)
 		)
-		(pin "UART TXD" input
+		(pin "UART (TXD)" input
 			(at 137.16 67.31 270)
 			(effects
@@
 			)
 		)
-		(pin "power_on_pulse" input
+		(pin "power-on_pulse" input
 			(at 144.78 67.31 270)
 			(effects
@@
 			)
 		)
-		(pin "AT UART (RXD)" input
+		(pin "UART (RXD)" input
 			(at 134.62 78.74 90)
 			(effects
@@
 			)
 		)
-		(pin "AT UART (TXD)" input
+		(pin "UART (TXD)" input
 			(at 137.16 78.74 90)
 			(effects
@@
 			)
 		)
-		(pin "Battery_voltage_sense" input
+		(pin "battery_voltage_sense" input
 			(at 142.24 78.74 90)
 			(effects
@@
 				)
 				(justify left)
+			)
+		)
+		(pin "LED DIN" input
+			(at 199.39 106.68 0)
+			(effects
+				(font
+					(size 1.27 1.27)
+				)
+				(justify right)
 			)
 		)
@@
 				)
 			)
+		)
+	)
+	(sheet
+		(at 215.9 115.57)
+		(size 49.53 25.4)
+		(exclude_from_sim no)
+		(in_bom yes)
+		(on_board yes)
+		(dnp no)
+		(fields_autoplaced yes)
+		(stroke
+			(width 0.1524)
+			(type solid)
+		)
+		(fill
+			(color 0 0 0 0)
+		)
+		(property "Sheetname" "Visual"
+			(at 215.9 114.8584 0)
+			(show_name no)
+			(do_not_autoplace no)
+			(effects
+				(font
+					(size 1.27 1.27)
+				)
+				(justify left bottom)
+			)
+		)
+		(property "Sheetfile" "visual.kicad_sch"
+			(at 215.9 141.5546 0)
+			(show_name no)
+			(do_not_autoplace no)
+			(effects
+				(font
+					(size 1.27 1.27)
+				)
+				(justify left top)
+			)
+		)
+		(pin "LED_DIN" input
+			(at 215.9 116.84 180)
+			(effects
+				(font
+					(size 1.27 1.27)
+				)
+				(justify left)
+			)
+		)
+		(instances
+			(project "panic_button_tiny"
+				(path "/c4eb92e9-b42f-4db0-b1d9-0ef70f7ca601"
+					(page "10")
+				)
+			)

Commit message: [UPDATE] connections in the circuit schematic
Other:
- sheet brains ports: added LED_DIN; removed LED DIN
Changed lines of the file:
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@@
 			)
 		)
-		(pin "LED DIN" input
+		(pin "LED_DIN" input
 			(at 199.39 106.68 0)
 			(effects

Commit message: [UPDATE] the schematic wirering
Other:
- sheet Sound ports: added none; removed Buzzer-
- sheet brains ports: added Buzzer+; removed none
- sheet radio_layout ports: added BLE_ant_in; removed none
Changed lines of the file:
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@@
+	(wire
+		(pts
+			(xy 181.61 115.57) (xy 181.61 107.95)
+		)
+		(stroke
+			(width 0)
+			(type default)
+		)
+	)
 	(wire
 		(pts
@@
 			)
 		)
+		(pin "Buzzer+" input
+			(at 181.61 107.95 270)
+			(effects
+				(font
+					(size 1.27 1.27)
+				)
+				(justify left)
+			)
+		)
 		(instances
 			(project "panic_button_tiny"
@@
 		)
 		(pin "Buzzer+" input
-			(at 152.4 115.57 90)
-			(effects
-				(font
-					(size 1.27 1.27)
-				)
-				(justify right)
-			)
-		)
-		(pin "Buzzer-" input
-			(at 154.94 115.57 90)
+			(at 181.61 115.57 90)
 			(effects
 				(font
@@
 			)
 		)
+		(pin "BLE_ant_in" input
+			(at 215.9 95.25 180)
+			(effects
+				(font
+					(size 1.27 1.27)
+				)
+				(justify left)
+			)
+		)
