File: KiCad/v2/tiny/panic_button_tiny/li-ion_charging_handling.kicad_sch (KiCad schematic)
At the start: 19 parts, among them Q1 Si2305CDS, SW4 SPDT_Slide_SMD_6.7x2.6mm, U6 TP4056-42-ESOP8, U7 DW01A, U8 8205A

Commit message: [UPDATE] the schematic wirering
Parts:
- renumbered TP10 to TP1, TP12 to TP2, TP11 to TP3, TP13 to TP4, TP7 to TP5, TP8 to TP6, TP9 to TP7, U7 to U6, U8 to U7, U6 to U8
Other:
- moved on the sheet: LED1, LED2, Q1, R6, R7, R8, R9, SW4, TP5, TP6, TP7, U8

Commit message: [UPDATE] connections in the schematic to better represent the logic flow
Parts:
- added R6, R7: 470k_0603, PCM_Resistor_SMD_AKL:R_0603_1608Metric_Pad0.98x0.95mm_HandSolder, symbol PCM_4ms_Resistor:470k_0603
- renumbered R8 to R10, R9 to R11, R6 to R8, R7 to R9

Commit message: [UPDATE] the schematic with the connections
Parts:
- renumbered R8 to R10, R9 to R11, R10 to R12, R11 to R13, R6 to R8, R7 to R9
Changed lines of the file:
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@@
 		(dnp no)
 		(fields_autoplaced yes)
-		(property "Reference" "R6"
+		(property "Reference" "R8"
 			(at 114.3 59.6899 0)
 			(show_name no)
@@
 			(project "panic_button_tiny"
 				(path "/c4eb92e9-b42f-4db0-b1d9-0ef70f7ca601/bf7d15b7-3a35-46fb-a5a6-5ea810f2dc2c/4988fc48-ac14-475f-a329-fd119eb80de7"
-					(reference "R6")
+					(reference "R8")
 					(unit 1)
 				)
@@
 		(dnp no)
 		(fields_autoplaced yes)
-		(property "Reference" "R9"
+		(property "Reference" "R11"
 			(at 166.37 60.96 90)
 			(show_name no)
@@
 			(project "panic_button_tiny"
 				(path "/c4eb92e9-b42f-4db0-b1d9-0ef70f7ca601/bf7d15b7-3a35-46fb-a5a6-5ea810f2dc2c/4988fc48-ac14-475f-a329-fd119eb80de7"
-					(reference "R9")
+					(reference "R11")
 					(unit 1)
 				)
@@
 		(dnp no)
 		(fields_autoplaced yes)
-		(property "Reference" "R11"
+		(property "Reference" "R13"
 			(at 208.28 58.4199 0)
 			(show_name no)
@@
 			(project "panic_button_tiny"
 				(path "/c4eb92e9-b42f-4db0-b1d9-0ef70f7ca601/bf7d15b7-3a35-46fb-a5a6-5ea810f2dc2c/4988fc48-ac14-475f-a329-fd119eb80de7"
-					(reference "R11")
+					(reference "R13")
 					(unit 1)
 				)
@@
 		(dnp no)
 		(fields_autoplaced yes)
-		(property "Reference" "R7"
+		(property "Reference" "R9"
 			(at 120.65 50.7999 0)
 			(show_name no)
@@
 			(project "panic_button_tiny"
 				(path "/c4eb92e9-b42f-4db0-b1d9-0ef70f7ca601/bf7d15b7-3a35-46fb-a5a6-5ea810f2dc2c/4988fc48-ac14-475f-a329-fd119eb80de7"
-					(reference "R7")
+					(reference "R9")
 					(unit 1)
 				)
@@
 		(dnp no)
 		(fields_autoplaced yes)
-		(property "Reference" "R8"
+		(property "Reference" "R10"
 			(at 166.37 45.72 90)
 			(show_name no)
@@
 			(project "panic_button_tiny"
 				(path "/c4eb92e9-b42f-4db0-b1d9-0ef70f7ca601/bf7d15b7-3a35-46fb-a5a6-5ea810f2dc2c/4988fc48-ac14-475f-a329-fd119eb80de7"
-					(reference "R8")
+					(reference "R10")
 					(unit 1)
 				)
@@
 		(dnp no)
 		(fields_autoplaced yes)
-		(property "Reference" "R10"
+		(property "Reference" "R12"
 			(at 198.12 58.4199 0)
 			(show_name no)
@@
 			(project "panic_button_tiny"
 				(path "/c4eb92e9-b42f-4db0-b1d9-0ef70f7ca601/bf7d15b7-3a35-46fb-a5a6-5ea810f2dc2c/4988fc48-ac14-475f-a329-fd119eb80de7"
-					(reference "R10")
+					(reference "R12")
 					(unit 1)
 				)
