File: KiCad/v2/tiny/panic_button_tiny/uart.kicad_sch (KiCad schematic)
At the start: 9 parts, among them J3 PINHD_1x6_Male

Commit message: [UPDATE] connections in the schematic to better represent the logic flow
Parts:
- renumbered R10 to R12, R11 to R13
Changed lines of the file:
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@@
 		(in_pos_files yes)
 		(dnp no)
-		(property "Reference" "R11"
+		(property "Reference" "R13"
 			(at 44.45 21.844 90)
 			(show_name no)
@@
 			(project "panic_button_tiny"
 				(path "/c4eb92e9-b42f-4db0-b1d9-0ef70f7ca601/525ab16f-d6f3-4728-a011-f4f1ced9fd5e/6bd96638-a0ba-4dc0-955f-d7671e306c1b"
-					(reference "R11")
+					(reference "R13")
 					(unit 1)
 				)
@@
 		(in_pos_files yes)
 		(dnp no)
-		(property "Reference" "R10"
+		(property "Reference" "R12"
 			(at 36.83 19.304 90)
 			(show_name no)
@@
 			(project "panic_button_tiny"
 				(path "/c4eb92e9-b42f-4db0-b1d9-0ef70f7ca601/525ab16f-d6f3-4728-a011-f4f1ced9fd5e/6bd96638-a0ba-4dc0-955f-d7671e306c1b"
-					(reference "R10")
+					(reference "R12")
 					(unit 1)
 				)
@@
 		(in_pos_files yes)
 		(dnp no)
-		(property "Reference" "#PWR070"
+		(property "Reference" "#PWR073"
 			(at 36.83 19.05 0)
 			(hide yes)
@@
 			(project "panic_button_tiny"
 				(path "/c4eb92e9-b42f-4db0-b1d9-0ef70f7ca601/525ab16f-d6f3-4728-a011-f4f1ced9fd5e/6bd96638-a0ba-4dc0-955f-d7671e306c1b"
-					(reference "#PWR070")
+					(reference "#PWR073")
 					(unit 1)
 				)
@@
 		(in_pos_files yes)
 		(dnp no)
-		(property "Reference" "#PWR071"
+		(property "Reference" "#PWR074"
 			(at 26.67 21.59 0)
 			(hide yes)
@@
 			(project "panic_button_tiny"
 				(path "/c4eb92e9-b42f-4db0-b1d9-0ef70f7ca601/525ab16f-d6f3-4728-a011-f4f1ced9fd5e/6bd96638-a0ba-4dc0-955f-d7671e306c1b"
-					(reference "#PWR071")
-					(unit 1)
-				)
+					(reference "#PWR074")
+					(unit 1)
+				)

Commit message: [UPDATE] the schematic with the connections
Parts:
- renumbered R12 to R14, R13 to R15
Changed lines of the file:
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@@
 		(in_pos_files yes)
 		(dnp no)
-		(property "Reference" "R13"
+		(property "Reference" "R15"
 			(at 44.45 21.844 90)
 			(show_name no)
@@
 			(project "panic_button_tiny"
 				(path "/c4eb92e9-b42f-4db0-b1d9-0ef70f7ca601/525ab16f-d6f3-4728-a011-f4f1ced9fd5e/6bd96638-a0ba-4dc0-955f-d7671e306c1b"
-					(reference "R13")
+					(reference "R15")
 					(unit 1)
 				)
@@
 		(in_pos_files yes)
 		(dnp no)
-		(property "Reference" "R12"
+		(property "Reference" "R14"
 			(at 36.83 19.304 90)
 			(show_name no)
@@
 			(project "panic_button_tiny"
 				(path "/c4eb92e9-b42f-4db0-b1d9-0ef70f7ca601/525ab16f-d6f3-4728-a011-f4f1ced9fd5e/6bd96638-a0ba-4dc0-955f-d7671e306c1b"
-					(reference "R12")
+					(reference "R14")
 					(unit 1)
 				)
